File: antena-wifi.kicad_pcb (KiCad board)
At the start: 2 copper layers, 40.6 x 52.3 mm, 19 parts, among them J1 Conn_01x01, J2 USB_C_Receptacle_USB2.0, SW1 Sw_Res

Commit message: update płytki
Parts:
- G***: moved to B.Cu
- moved G*** 52.0 mm to (117.7, 151.5), turned to 180 degrees
Routing:
- net GND: track 42.7 -> 47.9 mm
- net Net-(J2-SHIELD): vias 6 -> 4
- added copper zone on F.Cu, net GND
Other:
- board text added: "BL-M8812EU2 LR comm board rev 1.0 04.09.2026 AGH Drone Engineering"
- board text added: "SW1"
- board text removed: "IMAV antenna PCB"
